Commit message: Fix: Nested git repositories removed, uploading full source code

File: cobot_description/urdf/base.urdf.xacro (robot description, xacro)
@@ -31,3 +31,6 @@
         <child link="base_link" />
     </joint>
+    <gazebo reference="base_link">
+        <material>Gazebo/White</material>
+    </gazebo>
 </robot>

File: cobot_description/urdf/finger.urdf.xacro (robot description, xacro)
@@ -68,3 +68,9 @@
         <limit lower="0.0" upper="0.025" effort="1000000" velocity="1000000" />
     </joint>
+    <gazebo reference="finger-1-link">
+        <material>Gazebo/SkyBlue</material>
+    </gazebo>
+    <gazebo reference="finger-2-link">
+        <material>Gazebo/SkyBlue</material>
+    </gazebo>
 </robot>

File: cobot_description/urdf/gripper.urdf.xacro (robot description, xacro)
@@ -33,3 +33,6 @@
         <child link="gripper-base-link" />
     </joint>
+    <gazebo reference="gripper-base-link">
+        <material>Gazebo/White</material>
+    </gazebo>
 </robot>

File: cobot_description/urdf/part-1.urdf.xacro (robot description, xacro)
@@ -33,3 +33,6 @@
         <axis xyz="0.0 0.0 1.0" />
     </joint>
+    <gazebo reference="part-1-link">
+        <material>Gazebo/SkyBlue</material>
+    </gazebo>
 </robot>

File: cobot_description/urdf/part-2.urdf.xacro (robot description, xacro)
@@ -34,3 +34,6 @@
         <axis xyz="-2.627434620609032e-46 -3.9443045261049027e-31 1.0" />
     </joint>
+     <gazebo reference="part-2-link">
+        <material>Gazebo/White</material>
+    </gazebo>
 </robot>

File: cobot_description/urdf/part-3.urdf.xacro (robot description, xacro)
@@ -33,3 +33,6 @@
         <axis xyz="-3.1529215447308384e-45 -1.0 -3.155443620884051e-30" />
     </joint>
+    <gazebo reference="part-3-link">
+        <material>Gazebo/SkyBlue</material>
+    </gazebo>
 </robot>

File: cobot_description/urdf/part-4.urdf.xacro (robot description, xacro)
@@ -34,3 +34,6 @@
         <axis xyz="0.0 0.0 1.0" />
     </joint>
+     <gazebo reference="part-2-link">
+        <material>Gazebo/White</material>
+    </gazebo>
 </robot>

File: cobot_description/urdf/part-5.urdf.xacro (robot description, xacro)
@@ -34,3 +34,6 @@
         <axis xyz="0.0 1.0 1.232595164407831e-32" />
     </joint>
+    <gazebo reference="part-3-link">
+        <material>Gazebo/SkyBlue</material>
+    </gazebo>
 </robot>

File: cobot_description/urdf/part-6.urdf.xacro (robot description, xacro)
@@ -34,3 +34,6 @@
         <axis xyz="9.55405697163452e-31 -1.0 -6.310887241768095e-30" />
     </joint>
+     <gazebo reference="part-2-link">
+        <material>Gazebo/White</material>
+    </gazebo>
 </robot>

File: cobot_description/urdf/ros2_control.xacro (robot description, xacro)
@@ -3,7 +3,5 @@
     <gazebo>
         <plugin name="gazebo_ros2_control" filename="libgazebo_ros2_control.so">
-            <parameters>
-                $(find cobot_control)/config/cobat_controller.yaml
-            </parameters>
+            <parameters>$(find cobot_moveit_config)/config/ros2_controllers.yaml</parameters>
         </plugin>
     </gazebo>
@@ -15,32 +13,40 @@
             <command_interface name="position" />
             <state_interface name="position" />
+            <state_interface name="velocity" />
         </joint>
         <joint name="part-2-joint">
             <command_interface name="position" />
             <state_interface name="position" />
+            <state_interface name="velocity" />
         </joint>
         <joint name="part-3-joint">
             <command_interface name="position" />
             <state_interface name="position" />
+            <state_interface name="velocity" />
         </joint>
         <joint name="part-4-joint">
             <command_interface name="position" />
             <state_interface name="position" />
+            <state_interface name="velocity" />
         </joint>
         <joint name="part-5-joint">
             <command_interface name="position" />
             <state_interface name="position" />
+            <state_interface name="velocity" />
         </joint>
         <joint name="part-6-joint">
             <command_interface name="position" />
             <state_interface name="position" />
+            <state_interface name="velocity" />
         </joint>
         <joint name="finger-1-joint">
             <command_interface name="position" />
             <state_interface name="position" />
+            <state_interface name="velocity" />
         </joint>
         <joint name="finger-2-joint">
             <command_interface name="position" />
             <state_interface name="position" />
+            <state_interface name="velocity" />
         </joint>
     </ros2_control>
